File: Hardware/Sahara.kicad_pcb (KiCad board)
At the start: 2 copper layers, 58 parts, among them K1 G6DN-1A-L_DC5, K2 G6DN-1A-L_DC5, Q1 BC847, Q2 BC847, U1 STM32F103CBT6, U2 AZ1117-3.3, U3 74HC595, U4 74HC595, U5 74HC595, U6 74HC595, U7 74HC595, U8 4N35, U9 4N35, Y1 8MHz 18 pF, Y2 32.768 7 pF

Commit message: Added temperature sensor and I2C setup, started PCB layout
Parts:
- removed C10, C11: 10p, Capacitor_SMD:C_0805_2012Metric
- removed Y2: 32.768 7 pF, SamacSys_Parts:SC32S7PF20PPM
- added D1: BAS70-04, SamacSys_Parts:SOT97P230X109-3N, B.Cu at (54.2, 89.3)
- added D2: BAS70-04, SamacSys_Parts:SOT97P230X109-3N, B.Cu at (54.2, 93.9)
- added F1: 2A, SamacSys_Parts:WR-FSH_THT_2, B.Cu at (156.0, 129.0)
- added J1: Conn_01x02, TerminalBlock_Phoenix:TerminalBlock_Phoenix_PT-1,5-2-5.0-H_1x02_P5.00mm_Horizontal, B.Cu at (177.2, 128.8)
- added J2: TMP102_CONN, Connector_JST:JST_XH_B4B-XH-AM_1x04_P2.50mm_Vertical, B.Cu at (223.8, 109.8)
- added J3: Conn_01x02, Connector_JST:JST_XH_B2B-XH-AM_1x02_P2.50mm_Vertical, B.Cu at (106.8, 88.0)
- added J4: Conn_01x04, Connector_JST:JST_XH_B4B-XH-AM_1x04_P2.50mm_Vertical, F.Cu at (159.5, 87.2)
- added J6: Conn_01x02, TerminalBlock_Phoenix:TerminalBlock_Phoenix_PT-1,5-2-5.0-H_1x02_P5.00mm_Horizontal, B.Cu at (106.5, 128.8)
- added LED1: RGB_LED, SamacSys_Parts:5218559F, F.Cu at (101.9, 94.0)
- added R18: 150, Resistor_SMD:R_0805_2012Metric, F.Cu at (84.7, 67.3)
- added R19: 80, Resistor_SMD:R_0805_2012Metric, F.Cu at (84.7, 70.2)
- added R20: 80, Resistor_SMD:R_0805_2012Metric, F.Cu at (84.7, 73.2)
- added R21: 4.7k, Resistor_SMD:R_0805_2012Metric, F.Cu at (91.1, 67.3)
- added R22: 4.7k, Resistor_SMD:R_0805_2012Metric, F.Cu at (91.1, 70.2)
- added REF**: Symbol_HighVoltage_Triangle_6x6mm_Copper, Symbol:Symbol_HighVoltage_Triangle_6x6mm_Copper, F.Cu at (134.0, 120.9)
- added REF**: Symbol_HighVoltage_Triangle_6x6mm_Copper, Symbol:Symbol_HighVoltage_Triangle_6x6mm_Copper, B.Cu at (189.5, 120.2)
- Q1, Q2, R10, R11, R12, R13, R14, R15, U8, U9: moved to B.Cu
- moved Q1 181.7 mm to (47.3, 101.8), turned to 180 degrees
- moved Q2 181.7 mm to (47.3, 106.4), turned to 180 degrees
- moved R10 181.7 mm to (21.8, 100.9), turned to 180 degrees
- moved R11 181.7 mm to (21.8, 103.8), turned to 180 degrees
- moved R12 181.7 mm to (21.8, 106.8), turned to 180 degrees
- moved R13 181.7 mm to (21.8, 109.7), turned to 180 degrees
- moved R14 181.7 mm to (21.8, 112.7), turned to 180 degrees
- moved R15 181.7 mm to (21.8, 115.6), turned to 180 degrees
- moved U8 181.7 mm to (29.2, 106.1), turned to 180 degrees
- moved R7 178.7 mm to (99.8, 114.6), turned to 90 degrees
- moved R9 157.7 mm to (120.0, 114.6), turned to -90 degrees
- moved R8 155.7 mm to (120.2, 101.9), turned to -90 degrees
- moved C13 147.1 mm to (123.1, 88.0), turned to -90 degrees
- moved VR1 145.4 mm to (107.2, 115.5)
- moved U2 139.9 mm to (115.8, 89.0), turned to 90 degrees
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Connections:
- K1 pad 5: FAN_LIVE -> 230v AC
- K1 pad 8: 230v AC -> FAN_LIVE
- K2 pad 5: HEATER_LIVE -> 230v AC
- K2 pad 8: 230v AC -> HEATER_LIVE
- RN1 pad 1: unconnected-(RN1-R1.1-Pad1) -> Net-(DS1-B)
- RN1 pad 10: Net-(DS1-D) -> Net-(RN1-R7.2)
- RN1 pad 11: Net-(DS1-C) -> Net-(RN1-R6.2)
- RN1 pad 12: Net-(DS1-G) -> Net-(RN1-R5.2)
- RN1 pad 13: Net-(DS1-F) -> Net-(RN1-R4.2)
- RN1 pad 14: Net-(DS1-A) -> Net-(RN1-R3.2)
- RN1 pad 15: Net-(DS1-B) -> Net-(RN1-R2.2)
- RN1 pad 16: unconnected-(RN1-R1.2-Pad16) -> Net-(RN1-R1.2)
- RN1 pad 2: Net-(RN1-R2.1) -> Net-(DS1-A)
- RN1 pad 3: Net-(RN1-R3.1) -> Net-(DS1-F)
- RN1 pad 4: Net-(RN1-R4.1) -> Net-(DS1-G)
- RN1 pad 5: Net-(RN1-R5.1) -> Net-(DS1-C)
- RN1 pad 6: Net-(RN1-R6.1) -> Net-(DS1-D)
- RN1 pad 7: Net-(RN1-R7.1) -> Net-(DS1-E)
- RN1 pad 8: Net-(RN1-R8.1) -> unconnected-(RN1-R8.1-Pad8)
- RN1 pad 9: Net-(DS1-E) -> unconnected-(RN1-R8.2-Pad9)
- RN2 pad 10: Net-(DS2-D) -> Net-(RN2-R7.2)
- RN2 pad 11: Net-(DS2-C) -> Net-(RN2-R6.2)
- RN2 pad 12: Net-(DS2-G) -> Net-(RN2-R5.2)
- RN2 pad 13: Net-(DS2-F) -> Net-(RN2-R4.2)
- RN2 pad 14: Net-(DS2-A) -> Net-(RN2-R3.2)
- RN2 pad 15: Net-(DS2-B) -> Net-(RN2-R2.2)
- RN2 pad 2: Net-(RN2-R2.1) -> Net-(DS2-B)
- RN2 pad 3: Net-(RN2-R3.1) -> Net-(DS2-A)
- RN2 pad 4: Net-(RN2-R4.1) -> Net-(DS2-F)
- RN2 pad 5: Net-(RN2-R5.1) -> Net-(DS2-G)
- RN2 pad 6: Net-(RN2-R6.1) -> Net-(DS2-C)
- RN2 pad 7: Net-(RN2-R7.1) -> Net-(DS2-D)
- RN2 pad 8: Net-(RN2-R8.1) -> Net-(DS2-E)
- RN2 pad 9: Net-(DS2-E) -> Net-(RN2-R8.2)
- RN3 pad 1: Net-(RN3-R1.1) -> Net-(DS3-B)
- RN3 pad 10: Net-(DS3-E) -> Net-(RN3-R7.2)
- RN3 pad 11: Net-(DS3-D) -> Net-(RN3-R6.2)
- RN3 pad 12: Net-(DS3-C) -> Net-(RN3-R5.2)
- RN3 pad 13: Net-(DS3-G) -> Net-(RN3-R4.2)
- RN3 pad 14: Net-(DS3-F) -> Net-(RN3-R3.2)
- RN3 pad 15: Net-(DS3-A) -> Net-(RN3-R2.2)
- RN3 pad 16: Net-(DS3-B) -> Net-(RN3-R1.2)
- RN3 pad 2: Net-(RN3-R2.1) -> Net-(DS3-A)
- RN3 pad 3: Net-(RN3-R3.1) -> Net-(DS3-F)
- RN3 pad 4: Net-(RN3-R4.1) -> Net-(DS3-G)
- RN3 pad 5: Net-(RN3-R5.1) -> Net-(DS3-C)
- RN3 pad 6: Net-(RN3-R6.1) -> Net-(DS3-D)
- RN3 pad 7: Net-(RN3-R7.1) -> Net-(DS3-E)
- RN3 pad 8: +3.3V -> Net-(DS3-DP)
- RN3 pad 9: Net-(DS3-DP) -> +3.3V
- RN4 pad 10: Net-(DS4-D) -> Net-(RN4-R7.2)
- RN4 pad 11: Net-(DS4-C) -> Net-(RN4-R6.2)
- RN4 pad 12: Net-(DS4-G) -> Net-(RN4-R5.2)
- RN4 pad 13: Net-(DS4-F) -> Net-(RN4-R4.2)
- RN4 pad 14: Net-(DS4-A) -> Net-(RN4-R3.2)
- RN4 pad 15: Net-(DS4-B) -> Net-(RN4-R2.2)
- RN4 pad 2: Net-(RN4-R2.1) -> Net-(DS4-B)
- RN4 pad 3: Net-(RN4-R3.1) -> Net-(DS4-A)
- RN4 pad 4: Net-(RN4-R4.1) -> Net-(DS4-F)
- RN4 pad 5: Net-(RN4-R5.1) -> Net-(DS4-G)
- RN4 pad 6: Net-(RN4-R6.1) -> Net-(DS4-C)
- RN4 pad 7: Net-(RN4-R7.1) -> Net-(DS4-D)
- RN4 pad 8: Net-(RN4-R8.1) -> Net-(DS4-E)
- RN4 pad 9: Net-(DS4-E) -> Net-(RN4-R8.2)
- RN5 pad 10: Net-(DS5-D) -> Net-(RN5-R7.2)
- RN5 pad 11: Net-(DS5-C) -> Net-(RN5-R6.2)
- RN5 pad 12: Net-(DS5-G) -> Net-(RN5-R5.2)
- RN5 pad 13: Net-(DS5-F) -> Net-(RN5-R4.2)
- RN5 pad 14: Net-(DS5-A) -> Net-(RN5-R3.2)
- RN5 pad 15: Net-(DS5-B) -> Net-(RN5-R2.2)
- RN5 pad 2: Net-(RN5-R2.1) -> Net-(DS5-B)
- RN5 pad 3: Net-(RN5-R3.1) -> Net-(DS5-A)
- RN5 pad 4: Net-(RN5-R4.1) -> Net-(DS5-F)
- RN5 pad 5: Net-(RN5-R5.1) -> Net-(DS5-G)
- RN5 pad 6: Net-(RN5-R6.1) -> Net-(DS5-C)
- RN5 pad 7: Net-(RN5-R7.1) -> Net-(DS5-D)
- RN5 pad 8: Net-(RN5-R8.1) -> Net-(DS5-E)
- RN5 pad 9: Net-(DS5-E) -> Net-(RN5-R8.2)
- U1 pad 1: unconnected-(U1-VBAT-Pad1) -> +3.3V
- U1 pad 13: unconnected-(U1-PA3-Pad13) -> FAN_CONTROL
- U1 pad 14: unconnected-(U1-PA4-Pad14) -> HEATER_CONTROL
- U1 pad 3: OSC32_IN -> unconnected-(U1-PC14-Pad3)
- U1 pad 39: unconnected-(U1-PB3-Pad39) -> LED_GREEN
- U1 pad 4: OSC_OUT -> unconnected-(U1-PC15-Pad4)
- U1 pad 40: unconnected-(U1-PB4-Pad40) -> LED_BLUE
- U1 pad 41: unconnected-(U1-PB5-Pad41) -> LED_RED
- U1 pad 42: unconnected-(U1-PB6-Pad42) -> SCL
- U1 pad 43: FAN_CONTROL -> SDA
- U1 pad 45: HEATER_CONTROL -> unconnected-(U1-PB8-Pad45)
- U3 pad 1: Net-(RN1-R2.1) -> Net-(RN1-R1.2)
- U3 pad 2: Net-(RN1-R3.1) -> Net-(RN1-R2.2)
- U3 pad 3: Net-(RN1-R4.1) -> Net-(RN1-R3.2)
- U3 pad 4: Net-(RN1-R5.1) -> Net-(RN1-R4.2)
- U3 pad 5: Net-(RN1-R6.1) -> Net-(RN1-R5.2)
- U3 pad 6: Net-(RN1-R7.1) -> Net-(RN1-R6.2)
- U3 pad 7: Net-(RN1-R8.1) -> Net-(RN1-R7.2)
- U4 pad 1: Net-(RN2-R2.1) -> Net-(RN2-R2.2)
- U4 pad 2: Net-(RN2-R3.1) -> Net-(RN2-R3.2)
- U4 pad 3: Net-(RN2-R4.1) -> Net-(RN2-R4.2)
- U4 pad 4: Net-(RN2-R5.1) -> Net-(RN2-R5.2)
- U4 pad 5: Net-(RN2-R6.1) -> Net-(RN2-R6.2)
- U4 pad 6: Net-(RN2-R7.1) -> Net-(RN2-R7.2)
- U4 pad 7: Net-(RN2-R8.1) -> Net-(RN2-R8.2)
- U5 pad 1: Net-(RN3-R1.1) -> Net-(RN3-R1.2)
- U5 pad 2: Net-(RN3-R2.1) -> Net-(RN3-R2.2)
- U5 pad 3: Net-(RN3-R3.1) -> Net-(RN3-R3.2)
- U5 pad 4: Net-(RN3-R4.1) -> Net-(RN3-R4.2)
- U5 pad 5: Net-(RN3-R5.1) -> Net-(RN3-R5.2)
- U5 pad 6: Net-(RN3-R6.1) -> Net-(RN3-R6.2)
- U5 pad 7: Net-(RN3-R7.1) -> Net-(RN3-R7.2)
- U6 pad 1: Net-(RN4-R2.1) -> Net-(RN4-R2.2)
- U6 pad 2: Net-(RN4-R3.1) -> Net-(RN4-R3.2)
- U6 pad 3: Net-(RN4-R4.1) -> Net-(RN4-R4.2)
- U6 pad 4: Net-(RN4-R5.1) -> Net-(RN4-R5.2)
- U6 pad 5: Net-(RN4-R6.1) -> Net-(RN4-R6.2)
- U6 pad 6: Net-(RN4-R7.1) -> Net-(RN4-R7.2)
- U6 pad 7: Net-(RN4-R8.1) -> Net-(RN4-R8.2)
- U7 pad 1: Net-(RN5-R2.1) -> Net-(RN5-R2.2)
- U7 pad 2: Net-(RN5-R3.1) -> Net-(RN5-R3.2)
- U7 pad 3: Net-(RN5-R4.1) -> Net-(RN5-R4.2)
- U7 pad 4: Net-(RN5-R5.1) -> Net-(RN5-R5.2)
- U7 pad 5: Net-(RN5-R6.1) -> Net-(RN5-R6.2)
- U7 pad 6: Net-(RN5-R7.1) -> Net-(RN5-R7.2)
- U7 pad 7: Net-(RN5-R8.1) -> Net-(RN5-R8.2)
Routing:
- net +3.3V: track 0.00 -> 229.9 mm
- net 230v AC: track 0.00 -> 77.5 mm
- net FAN_LIVE: track 0.00 -> 16.9 mm
- net MOSI: track 0.00 -> 16.4 mm
- net OSC_OUT: track 0.00 -> 13.4 mm
- net OSC_IN: track 0.00 -> 13.4 mm
- net SWCLK: track 0.00 -> 11.4 mm, vias 0 -> 1
- net +5V: track 0.00 -> 11.3 mm
- net SCK: track 0.00 -> 11.0 mm
- net TimeLatch: track 0.00 -> 9.07 mm
- net EncBut: track 0.00 -> 8.00 mm
- net TIM1_CH2: track 0.00 -> 7.75 mm
- net TIM1_CH1: track 0.00 -> 7.50 mm
- net Net-(U1-NRST): track 0.00 -> 7.28 mm
- net HEATER_LIVE: track 0.00 -> 7.17 mm
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- added copper zone on B.Cu, net Earth
- added copper zone on F.Cu, net Earth
Other:
- board outline added: 130 x 50 mm
- board text added: "23/03/2025"
- board text added: "DANGER HIGH VOlTAGE"
- board text added: "SAHARA"
- board text added: "V1.0 - Acrylic"

Commit message: Software stuff
Connections:
- U1 pad 13: FAN_CONTROL -> HEATER_CONTROL
- U1 pad 14: HEATER_CONTROL -> unconnected-(U1-PA4-Pad14)
- U1 pad 20: unconnected-(U1-PB2-Pad20) -> TimeLatch
- U1 pad 46: TimeLatch -> FAN_CONTROL

Commit message: Almost finished PCB
Parts:
- R18, R19, R20: moved to B.Cu
- moved R15 186.3 mm to (208.0, 108.1), turned to 90 degrees
- moved R13 178.6 mm to (200.4, 106.5), turned to 0 degrees
- moved R11 161.6 mm to (183.3, 108.2), turned to 90 degrees
- moved Q2 157.6 mm to (204.9, 108.2)
- moved D2 151.9 mm to (204.9, 112.9), turned to 0 degrees
- moved R21 137.6 mm to (225.5, 96.6), turned to -90 degrees
- moved R22 133.4 mm to (221.9, 96.6), turned to -90 degrees
- moved R10 119.3 mm to (141.1, 105.6), turned to 0 degrees
- moved U8 102.9 mm to (132.1, 108.1), turned to -90 degrees
- moved R12 102.7 mm to (124.5, 108.2), turned to 90 degrees
- moved R14 99.4 mm to (121.0, 105.3), turned to 0 degrees
- moved Q1 73.9 mm to (121.0, 108.2)
- moved D1 70.8 mm to (121.0, 112.9), turned to 0 degrees
- moved U9 62.3 mm to (192.3, 109.0), turned to 90 degrees
- moved R18 41.1 mm to (113.1, 97.1)
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Connections:
- RN1 pad 1: Net-(DS1-B) -> Net-(DS1-E)
- RN1 pad 2: Net-(DS1-A) -> Net-(DS1-D)
- RN1 pad 3: Net-(DS1-F) -> Net-(DS1-C)
- RN1 pad 5: Net-(DS1-C) -> Net-(DS1-F)
- RN1 pad 6: Net-(DS1-D) -> Net-(DS1-A)
- RN1 pad 7: Net-(DS1-E) -> Net-(DS1-B)
- RN2 pad 1: unconnected-(RN2-R1.1-Pad1) -> Net-(DS2-E)
- RN2 pad 16: unconnected-(RN2-R1.2-Pad16) -> Net-(RN2-R1.2)
- RN2 pad 2: Net-(DS2-B) -> Net-(DS2-D)
- RN2 pad 3: Net-(DS2-A) -> Net-(DS2-C)
- RN2 pad 4: Net-(DS2-F) -> Net-(DS2-G)
- RN2 pad 5: Net-(DS2-G) -> Net-(DS2-F)
- RN2 pad 6: Net-(DS2-C) -> Net-(DS2-A)
- RN2 pad 7: Net-(DS2-D) -> Net-(DS2-B)
- RN2 pad 8: Net-(DS2-E) -> unconnected-(RN2-R8.1-Pad8)
- RN2 pad 9: Net-(RN2-R8.2) -> unconnected-(RN2-R8.2-Pad9)
- RN3 pad 1: Net-(DS3-B) -> Net-(DS3-E)
- RN3 pad 2: Net-(DS3-A) -> Net-(DS3-D)
- RN3 pad 3: Net-(DS3-F) -> Net-(DS3-C)
- RN3 pad 5: Net-(DS3-C) -> Net-(DS3-F)
- RN3 pad 6: Net-(DS3-D) -> Net-(DS3-A)
- RN3 pad 7: Net-(DS3-E) -> Net-(DS3-B)
- RN4 pad 1: unconnected-(RN4-R1.1-Pad1) -> Net-(DS4-E)
- RN4 pad 16: unconnected-(RN4-R1.2-Pad16) -> Net-(RN4-R1.2)
- RN4 pad 2: Net-(DS4-B) -> Net-(DS4-D)
- RN4 pad 3: Net-(DS4-A) -> Net-(DS4-C)
- RN4 pad 4: Net-(DS4-F) -> Net-(DS4-G)
- RN4 pad 5: Net-(DS4-G) -> Net-(DS4-F)
- RN4 pad 6: Net-(DS4-C) -> Net-(DS4-A)
- RN4 pad 7: Net-(DS4-D) -> Net-(DS4-B)
- RN4 pad 8: Net-(DS4-E) -> unconnected-(RN4-R8.1-Pad8)
- RN4 pad 9: Net-(RN4-R8.2) -> unconnected-(RN4-R8.2-Pad9)
- RN5 pad 1: unconnected-(RN5-R1.1-Pad1) -> Net-(DS5-E)
- RN5 pad 16: unconnected-(RN5-R1.2-Pad16) -> Net-(RN5-R1.2)
- RN5 pad 2: Net-(DS5-B) -> Net-(DS5-D)
- RN5 pad 3: Net-(DS5-A) -> Net-(DS5-C)
- RN5 pad 4: Net-(DS5-F) -> Net-(DS5-G)
- RN5 pad 5: Net-(DS5-G) -> Net-(DS5-F)
- RN5 pad 6: Net-(DS5-C) -> Net-(DS5-A)
- RN5 pad 7: Net-(DS5-D) -> Net-(DS5-B)
- RN5 pad 8: Net-(DS5-E) -> unconnected-(RN5-R8.1-Pad8)
- RN5 pad 9: Net-(RN5-R8.2) -> unconnected-(RN5-R8.2-Pad9)
- U1 pad 21: TempLatch -> unconnected-(U1-PB10-Pad21)
- U1 pad 32: unconnected-(U1-PA11-Pad32) -> TempLatch
- U4 pad 1: Net-(RN2-R2.2) -> Net-(RN2-R1.2)
- U4 pad 2: Net-(RN2-R3.2) -> Net-(RN2-R2.2)
- U4 pad 3: Net-(RN2-R4.2) -> Net-(RN2-R3.2)
- U4 pad 4: Net-(RN2-R5.2) -> Net-(RN2-R4.2)
- U4 pad 5: Net-(RN2-R6.2) -> Net-(RN2-R5.2)
- U4 pad 6: Net-(RN2-R7.2) -> Net-(RN2-R6.2)
- U4 pad 7: Net-(RN2-R8.2) -> Net-(RN2-R7.2)
- U6 pad 1: Net-(RN4-R2.2) -> Net-(RN4-R1.2)
- U6 pad 2: Net-(RN4-R3.2) -> Net-(RN4-R2.2)
- U6 pad 3: Net-(RN4-R4.2) -> Net-(RN4-R3.2)
- U6 pad 4: Net-(RN4-R5.2) -> Net-(RN4-R4.2)
- U6 pad 5: Net-(RN4-R6.2) -> Net-(RN4-R5.2)
- U6 pad 6: Net-(RN4-R7.2) -> Net-(RN4-R6.2)
- U6 pad 7: Net-(RN4-R8.2) -> Net-(RN4-R7.2)
- U7 pad 1: Net-(RN5-R2.2) -> Net-(RN5-R1.2)
- U7 pad 2: Net-(RN5-R3.2) -> Net-(RN5-R2.2)
- U7 pad 3: Net-(RN5-R4.2) -> Net-(RN5-R3.2)
- U7 pad 4: Net-(RN5-R5.2) -> Net-(RN5-R4.2)
- U7 pad 5: Net-(RN5-R6.2) -> Net-(RN5-R5.2)
- U7 pad 6: Net-(RN5-R7.2) -> Net-(RN5-R6.2)
- U7 pad 7: Net-(RN5-R8.2) -> Net-(RN5-R7.2)
Routing:
- net +5V: track 11.3 -> 227.9 mm
- net SCLR: track 0.00 -> 115.7 mm, vias 0 -> 7
- net SCK: track 11.0 -> 115.1 mm, vias 0 -> 6
- net +3.3V: track 229.9 -> 330.2 mm, vias 0 -> 1
- net TIM1_CH2: track 7.75 -> 103.2 mm, vias 0 -> 4
- net TIM1_CH1: track 7.50 -> 96.0 mm, vias 0 -> 2
- net SDA: track 0.00 -> 84.3 mm, vias 0 -> 1
- net SCL: track 0.00 -> 80.7 mm, vias 0 -> 1
- net MOSI: track 16.4 -> 71.7 mm, vias 0 -> 2
- net TimeLatch: track 9.07 -> 64.0 mm, vias 0 -> 2
- net TempLatch: track 0.00 -> 54.2 mm, vias 0 -> 3
- net EncBut: track 8.00 -> 60.4 mm, vias 0 -> 2
- net LED_GREEN: track 0.00 -> 48.4 mm, vias 0 -> 1
- net LED_BLUE: track 0.00 -> 47.9 mm, vias 0 -> 1
- net LED_RED: track 0.00 -> 47.6 mm, vias 0 -> 1
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