File: Hardware/Sahara.kicad_sch (KiCad schematic)
At the start: 24 parts, among them J3 Conn_01x02, J4 Conn_01x04, SW1 SW_Push, U1 STM32F103CBT6, U2 AZ1117-3.3, Y1 8MHz 18 pF

Commit message: Software stuff
Connections:
- net FAN_CONTROL: now also U1.46 (PB9); no longer U1.13 (PA3)
- net HEATER_CONTROL: now also U1.13 (PA3); no longer U1.14 (PA4)
- net TimeLatch: now also U1.20 (PB2); no longer U1.46 (PB9)
Other:
- moved on the sheet: R2
Changed lines of the file:
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@@
 	)
 	(junction
-		(at 41.91 99.06)
-		(diameter 0)
-		(color 0 0 0 0)
-	)
-	(junction
 		(at 125.73 60.96)
 		(diameter 0)
@@
 	)
 	(junction
+		(at 26.67 81.28)
+		(diameter 0)
+		(color 0 0 0 0)
+	)
+	(junction
 		(at 78.74 36.83)
 		(diameter 0)
@@
 	(wire
 		(pts
-			(xy 39.37 99.06) (xy 41.91 99.06)
+			(xy 24.13 81.28) (xy 26.67 81.28)
 		)
 		(stroke
@@
 	(wire
 		(pts
+			(xy 26.67 81.28) (xy 60.96 81.28)
+		)
+		(stroke
+			(width 0)
+			(type default)
+		)
+	)
+	(wire
+		(pts
 			(xy 73.66 43.18) (xy 73.66 40.64)
 		)
@@
 	(wire
 		(pts
-			(xy 97.79 36.83) (xy 102.87 36.83)
+			(xy 52.07 99.06) (xy 60.96 99.06)
 		)
 		(stroke
@@
 	(wire
 		(pts
-			(xy 73.66 40.64) (xy 76.2 40.64)
+			(xy 97.79 36.83) (xy 102.87 36.83)
 		)
 		(stroke
@@
 	(wire
 		(pts
-			(xy 81.28 43.18) (xy 81.28 40.64)
+			(xy 73.66 40.64) (xy 76.2 40.64)
 		)
 		(stroke
@@
 	(wire
 		(pts
-			(xy 93.98 68.58) (xy 97.79 68.58)
+			(xy 81.28 43.18) (xy 81.28 40.64)
 		)
 		(stroke
@@
 	(wire
 		(pts
-			(xy 33.02 76.2) (xy 60.96 76.2)
+			(xy 93.98 68.58) (xy 97.79 68.58)
 		)
 		(stroke
@@
 	(wire
 		(pts
-			(xy 57.15 36.83) (xy 78.74 36.83)
+			(xy 33.02 76.2) (xy 60.96 76.2)
 		)
 		(stroke
@@
 	(wire
 		(pts
-			(xy 36.83 48.26) (xy 43.18 48.26)
+			(xy 57.15 36.83) (xy 78.74 36.83)
 		)
 		(stroke
@@
 	(wire
 		(pts
-			(xy 41.91 99.06) (xy 60.96 99.06)
+			(xy 36.83 48.26) (xy 43.18 48.26)
 		)
 		(stroke
@@
 	(global_label "FAN_CONTROL"
 		(shape input)
-		(at 93.98 55.88 0)
+		(at 52.07 99.06 180)
 		(fields_autoplaced yes)
 		(effects
@@
 				(size 1.27 1.27)
 			)
-			(justify left)
+			(justify right)
 		)
 		(property "Intersheetrefs" "${INTERSHEET_REFS}"
-			(at 109.9677 55.88 0)
+			(at 36.0823 99.06 0)
 			(effects
 				(font
 					(size 1.27 1.27)
 				)
-				(justify left)
+				(justify right)
 				(hide yes)
 			)
@@
 	(global_label "TimeLatch"
 		(shape input)
-		(at 39.37 99.06 180)
+		(at 24.13 81.28 180)
 		(fields_autoplaced yes)
 		(effects
@@
 		)
 		(property "Intersheetrefs" "${INTERSHEET_REFS}"
-			(at 26.8901 99.06 0)
+			(at 11.6501 81.28 0)
 			(effects
 				(font
@@
 	(global_label "HEATER_CONTROL"
 		(shape input)
-		(at 93.98 58.42 0)
+		(at 93.98 55.88 0)
 		(fields_autoplaced yes)
 		(effects
@@
 		)
 		(property "Intersheetrefs" "${INTERSHEET_REFS}"
-			(at 113.4147 58.42 0)
+			(at 113.4147 55.88 0)
 			(effects
 				(font
@@
 	(symbol
 		(lib_id "power:Earth")
-		(at 41.91 106.68 0)
+		(at 26.67 88.9 0)
 		(mirror y)
 		(unit 1)
@@
 		(fields_autoplaced yes)
 		(property "Reference" "#PWR05"
-			(at 41.91 113.03 0)
+			(at 26.67 95.25 0)
 			(effects
 				(font
@@
 		)
 		(property "Value" "Earth"
-			(at 41.91 111.76 0)
+			(at 26.67 93.98 0)
 			(effects
 				(font
@@
 		)
 		(property "Footprint" ""
-			(at 41.91 106.68 0)
+			(at 26.67 88.9 0)
 			(effects
 				(font
@@
 		)
 		(property "Datasheet" "~"
-			(at 41.91 106.68 0)
+			(at 26.67 88.9 0)
 			(effects
 				(font
@@
 		)
 		(property "Description" "Power symbol creates a global label with name \"Earth\""
-			(at 41.91 106.68 0)
+			(at 26.67 88.9 0)
 			(effects
 				(font
@@
 		(on_board yes)
 		(dnp no)
-		(fields_autoplaced yes)
 		(property "Reference" "#PWR083"
 			(at 43.18 90.17 0)
@@
 		)
 		(property "Value" "+3.3V"
-			(at 43.18 81.28 0)
+			(at 42.926 82.55 0)
 			(effects
 				(font
@@
 		(on_board yes)
 		(dnp no)
-		(fields_autoplaced yes)
 		(property "Reference" "#PWR023"
 			(at 38.1 87.63 0)
@@
 		)
 		(property "Value" "+3.3V"
-			(at 38.1 78.74 0)
+			(at 38.354 79.756 0)
 			(effects
 				(font
@@
 	(symbol
 		(lib_id "Device:R_US")
-		(at 41.91 102.87 0)
+		(at 26.67 85.09 0)
 		(mirror y)
 		(unit 1)
@@
 		(fields_autoplaced yes)
 		(property "Reference" "R2"
-			(at 39.37 101.5999 0)
+			(at 24.13 83.8199 0)
 			(effects
 				(font
@@
 		)
 		(property "Value" "4.7k"
-			(at 39.37 104.1399 0)
+			(at 24.13 86.3599 0)
 			(effects
 				(font
@@
 		)
 		(property "Footprint" "Resistor_SMD:R_0805_2012Metric"
-			(at 40.894 103.124 90)
+			(at 25.654 85.344 90)
 			(effects
 				(font
@@
 		)
 		(property "Datasheet" "~"
-			(at 41.91 102.87 0)
+			(at 26.67 85.09 0)
 			(effects
 				(font
@@
 		)
 		(property "Description" "Resistor, US symbol"
-			(at 41.91 102.87 0)
+			(at 26.67 85.09 0)
 			(effects
 				(font

Commit message: Almost finished PCB
Connections:
- net TempLatch: now also U1.32 (PA11); no longer U1.21 (PB10)
Other:
- moved on the sheet: R3
Changed lines of the file:
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@@
-	)
-	(junction
-		(at 57.15 101.6)
-		(diameter 0)
-		(color 0 0 0 0)
 	)
 	(junction
@@
 	)
 	(junction
+		(at 111.76 82.55)
+		(diameter 0)
+		(color 0 0 0 0)
+	)
+	(junction
 		(at 33.02 76.2)
 		(diameter 0)
@@
 	(wire
 		(pts
+			(xy 111.76 76.2) (xy 111.76 82.55)
+		)
+		(stroke
+			(width 0)
+			(type default)
+		)
+	)
+	(wire
+		(pts
+			(xy 111.76 82.55) (xy 118.11 82.55)
+		)
+		(stroke
+			(width 0)
+			(type default)
+		)
+	)
+	(wire
+		(pts
 			(xy 43.18 48.26) (xy 60.96 48.26)
 		)
@@
 	(wire
 		(pts
+			(xy 93.98 76.2) (xy 111.76 76.2)
+		)
+		(stroke
+			(width 0)
+			(type default)
+		)
+	)
+	(wire
+		(pts
 			(xy 33.02 76.2) (xy 60.96 76.2)
 		)
@@
 	(wire
 		(pts
-			(xy 55.88 101.6) (xy 57.15 101.6)
-		)
-		(stroke
-			(width 0)
-			(type default)
-		)
-	)
-	(wire
-		(pts
 			(xy 81.28 40.64) (xy 78.74 40.64)
 		)
@@
 		(pts
 			(xy 166.37 30.48) (xy 166.37 29.21)
-		)
-		(stroke
-			(width 0)
-			(type default)
-		)
-	)
-	(wire
-		(pts
-			(xy 57.15 101.6) (xy 60.96 101.6)
 		)
 		(stroke
@@
 	(global_label "TempLatch"
 		(shape input)
-		(at 55.88 101.6 180)
+		(at 118.11 82.55 0)
 		(fields_autoplaced yes)
 		(effects
@@
 				(size 1.27 1.27)
 			)
-			(justify right)
+			(justify left)
 		)
 		(property "Intersheetrefs" "${INTERSHEET_REFS}"
-			(at 42.8559 101.6 0)
-			(effects
-				(font
-					(size 1.27 1.27)
-				)
-				(justify right)
+			(at 131.1341 82.55 0)
+			(effects
+				(font
+					(size 1.27 1.27)
+				)
+				(justify left)
 				(hide yes)
 			)
@@
 	(symbol
 		(lib_id "Device:R_US")
-		(at 57.15 105.41 0)
-		(mirror y)
+		(at 111.76 86.36 0)
 		(unit 1)
 		(exclude_from_sim no)
@@
 		(fields_autoplaced yes)
 		(property "Reference" "R3"
-			(at 54.61 104.1399 0)
+			(at 114.3 85.0899 0)
 			(effects
 				(font
@@
 		)
 		(property "Value" "4.7k"
-			(at 54.61 106.6799 0)
+			(at 114.3 87.6299 0)
 			(effects
 				(font
@@
 		)
 		(property "Footprint" "Resistor_SMD:R_0805_2012Metric"
-			(at 56.134 105.664 90)
+			(at 112.776 86.614 90)
 			(effects
 				(font
@@
 		)
 		(property "Datasheet" "~"
-			(at 57.15 105.41 0)
+			(at 111.76 86.36 0)
 			(effects
 				(font
@@
 		)
 		(property "Description" "Resistor, US symbol"
-			(at 57.15 105.41 0)
+			(at 111.76 86.36 0)
 			(effects
 				(font
@@
 	(symbol
 		(lib_id "power:Earth")
-		(at 57.15 109.22 0)
-		(mirror y)
+		(at 111.76 90.17 0)
 		(unit 1)
 		(exclude_from_sim no)
@@
 		(fields_autoplaced yes)
 		(property "Reference" "#PWR09"
-			(at 57.15 115.57 0)
+			(at 111.76 96.52 0)
 			(effects
 				(font
@@
 		)
 		(property "Value" "Earth"
-			(at 57.15 114.3 0)
+			(at 111.76 95.25 0)
 			(effects
 				(font
@@
 		)
 		(property "Footprint" ""
-			(at 57.15 109.22 0)
+			(at 111.76 90.17 0)
 			(effects
 				(font
@@
 		)
 		(property "Datasheet" "~"
-			(at 57.15 109.22 0)
+			(at 111.76 90.17 0)
 			(effects
 				(font
@@
 		)
 		(property "Description" "Power symbol creates a global label with name \"Earth\""
-			(at 57.15 109.22 0)
-			(effects
-				(font
+			(at 111.76 90.17 0)
+			(effects
+				(font

Commit message: slight schematic update, finished pcb(for now)
Parts:
- added R23: 10k, Resistor_SMD:R_0201_0603Metric, symbol Device:R_US
- SW1: footprint (none) -> Button_Switch_SMD:SW_Push_1P1T_NO_CK_KSC7xxJ
Connections:
- net Earth: now also R23.2
- net at U1.44 (BOOT0): now also R23.1
Other:
- moved on the sheet: C1, SW1
Changed lines of the file:
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@@
 	)
 	(junction
-		(at 43.18 48.26)
+		(at 35.56 48.26)
 		(diameter 0)
 		(color 0 0 0 0)
@@
 	(wire
 		(pts
+			(xy 48.26 53.34) (xy 60.96 53.34)
+		)
+		(stroke
+			(width 0)
+			(type default)
+		)
+	)
+	(wire
+		(pts
 			(xy 78.74 40.64) (xy 78.74 43.18)
 		)
@@
 	(wire
 		(pts
-			(xy 43.18 48.26) (xy 60.96 48.26)
+			(xy 35.56 48.26) (xy 60.96 48.26)
 		)
 		(stroke
@@
 	(wire
 		(pts
-			(xy 43.18 58.42) (xy 43.18 55.88)
+			(xy 35.56 58.42) (xy 35.56 55.88)
 		)
 		(stroke
@@
 	(wire
 		(pts
-			(xy 36.83 48.26) (xy 43.18 48.26)
+			(xy 29.21 48.26) (xy 35.56 48.26)
 		)
 		(stroke
@@
 	(symbol
 		(lib_id "Device:C")
-		(at 43.18 52.07 0)
+		(at 35.56 52.07 0)
 		(unit 1)
 		(exclude_from_sim no)
@@
 		(dnp no)
 		(property "Reference" "C1"
-			(at 46.228 51.054 0)
+			(at 38.608 51.054 0)
 			(effects
 				(font
@@
 		)
 		(property "Value" "100n"
-			(at 46.736 53.086 0)
+			(at 39.116 53.086 0)
 			(effects
 				(font
@@
 		)
 		(property "Footprint" "Capacitor_SMD:C_0805_2012Metric"
-			(at 44.1452 55.88 0)
+			(at 36.5252 55.88 0)
 			(effects
 				(font
@@
 		)
 		(property "Datasheet" "~"
-			(at 43.18 52.07 0)
+			(at 35.56 52.07 0)
 			(effects
 				(font
@@
 		)
 		(property "Description" "Unpolarized capacitor"
-			(at 43.18 52.07 0)
+			(at 35.56 52.07 0)
 			(effects
 				(font
@@
 	(symbol
 		(lib_id "power:Earth")
-		(at 36.83 58.42 0)
+		(at 29.21 58.42 0)
 		(mirror y)
 		(unit 1)
@@
 		(fields_autoplaced yes)
 		(property "Reference" "#PWR04"
-			(at 36.83 64.77 0)
+			(at 29.21 64.77 0)
 			(effects
 				(font
@@
 		)
 		(property "Value" "Earth"
-			(at 36.83 63.5 0)
+			(at 29.21 63.5 0)
 			(effects
 				(font
@@
 		)
 		(property "Footprint" ""
-			(at 36.83 58.42 0)
+			(at 29.21 58.42 0)
 			(effects
 				(font
@@
 		)
 		(property "Datasheet" "~"
-			(at 36.83 58.42 0)
+			(at 29.21 58.42 0)
 			(effects
 				(font
@@
 		)
 		(property "Description" "Power symbol creates a global label with name \"Earth\""
-			(at 36.83 58.42 0)
+			(at 29.21 58.42 0)
 			(effects
 				(font
@@
 	)
 	(symbol
+		(lib_id "power:Earth")
+		(at 48.26 60.96 0)
+		(mirror y)
+		(unit 1)
+		(exclude_from_sim no)
+		(in_bom yes)
+		(on_board yes)
+		(dnp no)
+		(fields_autoplaced yes)
+		(property "Reference" "#PWR086"
+			(at 48.26 67.31 0)
+			(effects
+				(font
+					(size 1.27 1.27)
+				)
+				(hide yes)
+			)
+		)
+		(property "Value" "Earth"
+			(at 48.26 66.04 0)
+			(effects
+				(font
+					(size 1.27 1.27)
+				)
+				(hide yes)
+			)
+		)
+		(property "Footprint" ""
+			(at 48.26 60.96 0)
+			(effects
+				(font
+					(size 1.27 1.27)
+				)
+				(hide yes)
+			)
+		)
+		(property "Datasheet" "~"
+			(at 48.26 60.96 0)
+			(effects
+				(font
+					(size 1.27 1.27)
+				)
+				(hide yes)
+			)
+		)
+		(property "Description" "Power symbol creates a global label with name \"Earth\""
+			(at 48.26 60.96 0)
+			(effects
+				(font
+					(size 1.27 1.27)
+				)
+				(hide yes)
+			)
+		)
+		(pin "1"
+		)
+		(instances
+			(project "Sahara"
+				(path "/1677429e-c497-4bfd-afaa-f24906fcbe1d"
+					(reference "#PWR086")
+					(unit 1)
+				)
+			)
+		)
+	)
+	(symbol
+		(lib_id "Device:R_US")
+		(at 48.26 57.15 0)
+		(mirror y)
+		(unit 1)
+		(exclude_from_sim no)
+		(in_bom yes)
+		(on_board yes)
+		(dnp no)
+		(property "Reference" "R23"
+			(at 45.72 55.8799 0)
+			(effects
+				(font
+					(size 1.27 1.27)
+				)
+				(justify left)
+			)
+		)
+		(property "Value" "10k"
+			(at 45.72 58.4199 0)
+			(effects
+				(font
+					(size 1.27 1.27)
+				)
+				(justify left)
+			)
+		)
+		(property "Footprint" "Resistor_SMD:R_0201_0603Metric"
+			(at 47.244 57.404 90)
+			(effects
+				(font
+					(size 1.27 1.27)
+				)
+				(hide yes)
+			)
+		)
+		(property "Datasheet" "~"
+			(at 48.26 57.15 0)
+			(effects
+				(font
+					(size 1.27 1.27)
+				)
+				(hide yes)
+			)
+		)
+		(property "Description" "Resistor, US symbol"
+			(at 48.26 57.15 0)
+			(effects
+				(font
+					(size 1.27 1.27)
+				)
+				(hide yes)
+			)
+		)
+		(pin "1"
+		)
+		(pin "2"
+		)
+		(instances
+			(project "Sahara"
+				(path "/1677429e-c497-4bfd-afaa-f24906fcbe1d"
+					(reference "R23")
+					(unit 1)
+				)
+			)
+		)
+	)
+	(symbol
 		(lib_id "Device:C")
 		(at 157.48 20.32 90)
@@
 	(symbol
 		(lib_id "power:Earth")
-		(at 43.18 58.42 0)
+		(at 35.56 58.42 0)
 		(mirror y)
 		(unit 1)
@@
 		(fields_autoplaced yes)
 		(property "Reference" "#PWR06"
-			(at 43.18 64.77 0)
+			(at 35.56 64.77 0)
 			(effects
 				(font
@@
 		)
 		(property "Value" "Earth"
-			(at 43.18 63.5 0)
+			(at 35.56 63.5 0)
 			(effects
 				(font
@@
 		)
 		(property "Footprint" ""
-			(at 43.18 58.42 0)
+			(at 35.56 58.42 0)
 			(effects
 				(font
@@
 		)
 		(property "Datasheet" "~"
-			(at 43.18 58.42 0)
+			(at 35.56 58.42 0)
 			(effects
 				(font
@@
 		)
 		(property "Description" "Power symbol creates a global label with name \"Earth\""
-			(at 43.18 58.42 0)
+			(at 35.56 58.42 0)
 			(effects
 				(font
@@
 	(symbol
 		(lib_id "Switch:SW_Push")
-		(at 36.83 53.34 90)
+		(at 29.21 53.34 90)
 		(unit 1)
 		(exclude_from_sim no)
@@
 		(dnp no)
 		(property "Reference" "SW1"
-			(at 25.4 51.562 90)
+			(at 17.78 51.562 90)
 			(effects
 				(font
@@
 		)
 		(property "Value" "SW_Push"
-			(at 25.4 54.102 90)
+			(at 17.78 54.102 90)
 			(effects
 				(font
@@
 			)
 		)
-		(property "Footprint" ""
-			(at 31.75 53.34 0)
+		(property "Footprint" "Button_Switch_SMD:SW_Push_1P1T_NO_CK_KSC7xxJ"
+			(at 24.13 53.34 0)
 			(effects
 				(font
@@
 		)
 		(property "Datasheet" "~"
-			(at 31.75 53.34 0)
+			(at 24.13 53.34 0)
 			(effects
 				(font
@@
 		)
 		(property "Description" "Push button switch, generic, two pins"
-			(at 36.83 53.34 0)
+			(at 29.21 53.34 0)
 			(effects
 				(font
