File: Hardware/UserInterface.kicad_sch (KiCad schematic)
At the start: 28 parts, among them U3 74HC595, U4 74HC595, U5 74HC595, U6 74HC595, U7 74HC595

Commit message: slight schematic update, finished pcb(for now)
Parts:
- removed RN1, RN2, RN3, RN4, RN5: 470, SamacSys_Parts:EXB2HV_1, symbol Device:R_Pack08
- added RN1, RN10, RN2, RN3, RN4, RN5, RN6, RN7, RN8, RN9: R_Pack04, Resistor_SMD:R_Array_Convex_4x1206, symbol Device:R_Pack04
Connections:
- net +3.3V: now also RN8.5 (R4.2)
- net at U7.1 (QB): now also RN5.8 (R1.2)
- net at U7.2 (QC): now also RN5.7 (R2.2)
- net at U7.3 (QD): now also RN5.6 (R3.2)
- net at U7.4 (QE): now also RN5.5 (R4.2)
- net at U7.5 (QF): now also RN10.8 (R1.2)
- net at U7.6 (QG): now also RN10.7 (R2.2)
- net at U7.7 (QH): now also RN10.6 (R3.2)
- net at U6.1 (QB): now also RN4.8 (R1.2)
- net at U6.2 (QC): now also RN4.7 (R2.2)
- net at U6.3 (QD): now also RN4.6 (R3.2)
- net at U6.4 (QE): now also RN4.5 (R4.2)
- net at U6.5 (QF): now also RN9.8 (R1.2)
- net at U6.6 (QG): now also RN9.7 (R2.2)
- net at U6.7 (QH): now also RN9.6 (R3.2)
- net at DS4.1 (E): now also RN4.1 (R1.1)
- net at DS4.10 (G): now also RN4.4 (R4.1)
- net at DS4.2 (D): now also RN4.2 (R2.1)
- net at DS4.4 (C): now also RN4.3 (R3.1)
- net at DS4.6 (B): now also RN9.3 (R3.1)
- net at DS4.7 (A): now also RN9.2 (R2.1)
- net at DS4.9 (F): now also RN9.1 (R1.1)
- net at DS2.1 (E): now also RN2.1 (R1.1)
- net at U4.7 (QH): now also RN7.6 (R3.2)
- net at U4.6 (QG): now also RN7.7 (R2.2)
- net at U4.5 (QF): now also RN7.8 (R1.2)
- net at U4.4 (QE): now also RN2.5 (R4.2)
- net at U4.3 (QD): now also RN2.6 (R3.2)
- net at U4.2 (QC): now also RN2.7 (R2.2)
- net at U4.1 (QB): now also RN2.8 (R1.2)
- net at DS2.2 (D): now also RN2.2 (R2.1)
- net at DS2.4 (C): now also RN2.3 (R3.1)
- net at DS2.10 (G): now also RN2.4 (R4.1)
- net at DS2.9 (F): now also RN7.1 (R1.1)
- net at DS2.7 (A): now also RN7.2 (R2.1)
- net at DS2.6 (B): now also RN7.3 (R3.1)
- net at DS5.1 (E): now also RN5.1 (R1.1)
- net at DS5.10 (G): now also RN5.4 (R4.1)
- net at DS5.2 (D): now also RN5.2 (R2.1)
- net at DS5.4 (C): now also RN5.3 (R3.1)
- net at DS5.6 (B): now also RN10.3 (R3.1)
- net at DS5.7 (A): now also RN10.2 (R2.1)
- net at DS5.9 (F): now also RN10.1 (R1.1)
- net at DS1.1 (E): now also RN6.1 (R1.1)
- net at U3.7 (QH): now also RN1.6 (R3.2)
- net at U3.6 (QG): now also RN1.7 (R2.2)
- net at U3.5 (QF): now also RN1.8 (R1.2)
- net at U3.4 (QE): now also RN6.5 (R4.2)
- net at U3.3 (QD): now also RN6.6 (R3.2)
- net at U3.2 (QC): now also RN6.7 (R2.2)
- net at U3.1 (QB): now also RN6.8 (R1.2)
- net at DS1.2 (D): now also RN6.2 (R2.1)
- net at DS1.4 (C): now also RN6.3 (R3.1)
- net at DS1.10 (G): now also RN6.4 (R4.1)
- net at DS1.9 (F): now also RN1.1 (R1.1)
- net at DS1.7 (A): now also RN1.2 (R2.1)
- net at DS1.6 (B): now also RN1.3 (R3.1)
- net at U5.1 (QB): now also RN3.8 (R1.2)
- net at U5.2 (QC): now also RN3.7 (R2.2)
- net at U5.3 (QD): now also RN3.6 (R3.2)
- net at U5.4 (QE): now also RN3.5 (R4.2)
- net at U5.5 (QF): now also RN8.8 (R1.2)
- net at U5.6 (QG): now also RN8.7 (R2.2)
- net at U5.7 (QH): now also RN8.6 (R3.2)
- net at DS3.1 (E): now also RN3.1 (R1.1)
- net at DS3.10 (G): now also RN3.4 (R4.1)
- net at DS3.2 (D): now also RN3.2 (R2.1)
- net at DS3.4 (C): now also RN3.3 (R3.1)
- net at DS3.5 (DP): now also RN8.4 (R4.1)
- net at DS3.6 (B): now also RN8.3 (R3.1)
- net at DS3.7 (A): now also RN8.2 (R2.1)
- net at DS3.9 (F): now also RN8.1 (R1.1)
