File: Hardware/_autosave-Sahara.kicad_pcb (KiCad board)
At the start: 2 copper layers, 130 x 50 mm, 78 parts, among them J1 Conn_01x02, J2 TMP102_CONN, J3 Conn_01x02, J4 Conn_01x04, J6 Conn_01x02, K1 G6DN-1A-L_DC5, K2 G6DN-1A-L_DC5, Q1 BC847, Q2 BC847, SW1 SW_Push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

Commit message: slight schematic update, finished pcb(for now)
Other:
- board text added: "28/03/2025"
- board text removed: "23/03/2025"
Changed lines of the file:
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@@
 		)
 	)
-	(gr_text "23/03/2025\n"
+	(gr_text "28/03/2025\n"
 		(at 212.75 132.25 0)
 		(layer "F.SilkS")
@@
 			(justify left bottom)
 		)
-		(render_cache "23/03/2025\n" 0
+		(render_cache "28/03/2025\n" 0
 			(polygon
 				(pts
@@
 			(polygon
 				(pts
-					(xy 214.57889 131.29158) (xy 214.416224 131.29158) (xy 214.416224 131.03366) (xy 214.57889 131.03366)
-					(xy 214.656857 131.027374) (xy 214.729586 131.004153) (xy 214.754745 130.988963) (xy 214.803342 130.931133)
-					(xy 214.817027 130.862934) (xy 214.801456 130.787005) (xy 214.754745 130.729944) (xy 214.685085 130.695495)
-					(xy 214.606482 130.6827) (xy 214.57889 130.68195) (xy 214.500851 130.686578) (xy 214.424117 130.699164)
-					(xy 214.39351 130.70613) (xy 214.31829 130.727081) (xy 214.247529 130.751718) (xy 214.188346 130.775739)
-					(xy 214.188346 130.494371) (xy 214.261 130.472852) (xy 214.332875 130.455142) (xy 214.39754 130.442348)
-					(xy 214.473617 130.431185) (xy 214.547428 130.425174) (xy 214.595376 130.42403) (xy 214.668776 130.426606)
-					(xy 214.749937 130.436497) (xy 214.823551 130.453808) (xy 214.899894 130.483381) (xy 214.965963 130.523051)
-					(xy 214.974563 130.529542) (xy 215.034029 130.58713) (xy 215.076504 130.654747) (xy 215.101989 130.732394)
-					(xy 215.110352 130.808561) (xy 215.110484 130.820069) (xy 215.102828 130.90019) (xy 215.079859 130.970651)
-					(xy 215.036906 131.037) (xy 215.032083 131.042452) (xy 214.976727 131.090659) (xy 214.908206 131.127203)
-					(xy 214.835279 131.150119) (xy 214.8086 131.155659) (xy 214.886132 131.174756) (xy 214.953864 131.203103)
-					(xy 215.018347 131.246051) (xy 215.059926 131.28755) (xy 215.101899 131.350559) (xy 215.130135 131.423769)
-					(xy 215.143702 131.497408) (xy 215.146755 131.557927) (xy 215.141718 131.638397) (xy 215.12661 131.711371)
-					(xy 215.096254 131.787032) (xy 215.052188 131.852491) (xy 215.003506 131.900478) (xy 214.934629 131.946444)
-					(xy 214.865712 131.976858) (xy 214.787677 131.998977) (xy 214.700522 132.012802) (xy 214.620927 132.017986)
-					(xy 214.587316 132.018447) (xy 214.507653 132.016282) (xy 214.428855 132.009789) (xy 214.357972 132.000129)
-					(xy 214.281564 131.985882) (xy 214.207492 131.967826) (xy 214.142184 131.948105) (xy 214.142184 131.666737)
-					(xy 214.210497 131.695667) (xy 214.282447 131.719489) (xy 214.351011 131.736713) (xy 214.429679 131.750271)
-					(xy 214.503524 131.757712) (xy 214.579588 131.760503) (xy 214.587316 131.760526) (xy 214.666138 131.753643)
-					(xy 214.7383 131.730433) (xy 214.782955 131.702274) (xy 214.832292 131.6432) (xy 214.854001 131.568557)
-					(xy 214.855129 131.544371) (xy 214.8466 131.467746) (xy 214.817844 131.398967) (xy 214.782955 131.357526)
-					(xy 214.720427 131.31734) (xy 214.648355 131.296796)
+					(xy 214.725597 130.427906) (xy 214.807931 130.442229) (xy 214.881604 130.467106) (xy 214.946617 130.502536)
+					(xy 214.987752 130.534305) (xy 215.042409 130.594252) (xy 215.08145 130.664181) (xy 215.104875 130.744094)
+					(xy 215.112561 130.822208) (xy 215.112683 130.833991) (xy 215.106851 130.907049) (xy 215.086965 130.978983)
+					(xy 215.052965 131.042086) (xy 215.000501 131.099599) (xy 214.938921 131.141368) (xy 214.878942 131.167749)
+					(xy 214.953381 131.198561) (xy 215.016873 131.241537) (xy 215.069416 131.296678) (xy 215.078611 131.309166)
+					(xy 215.116671 131.376564) (xy 215.140635 131.451905) (xy 215.15015 131.526502) (xy 215.150785 131.552798)
+					(xy 215.146186 131.632774) (xy 215.132392 131.70564) (xy 215.104675 131.781665) (xy 215.064441 131.848013)
+					(xy 215.019993 131.89718) (xy 214.957494 131.944432) (xy 214.884442 131.980077) (xy 214.813426 132.001394)
+					(xy 214.734656 132.014184) (xy 214.648133 132.018447) (xy 214.561858 132.014184) (xy 214.483286 132.001394)
+					(xy 214.412416 131.980077) (xy 214.339469 131.944432) (xy 214.277006 131.89718) (xy 214.226043 131.839127)
+					(xy 214.187597 131.771397) (xy 214.161669 131.69399) (xy 214.149407 131.619938) (xy 214.146214 131.552798)
+					(xy 214.147368 131.537411) (xy 214.420254 131.537411) (xy 214.429064 131.614416) (xy 214.458492 131.68435)
+					(xy 214.482903 131.716196) (xy 214.545544 131.762528) (xy 214.617147 131.782319) (xy 214.648133 131.783974)
+					(xy 214.724537 131.772606) (xy 214.792617 131.73494) (xy 214.813363 131.715097) (xy 214.8544 131.652544)
+					(xy 214.874516 131.57681) (xy 214.876744 131.537411) (xy 214.867883 131.460285) (xy 214.838283 131.39057)
+					(xy 214.813729 131.358991) (xy 214.751198 131.312909) (xy 214.67932 131.293226) (xy 214.648133 131.29158)
+					(xy 214.571552 131.302706) (xy 214.503552 131.339571) (xy 214.482903 131.358991) (xy 214.44234 131.420958)
+					(xy 214.422457 131.497315) (xy 214.420254 131.537411) (xy 214.147368 131.537411) (xy 214.15201 131.475524)
+					(xy 214.172045 131.397414) (xy 214.206392 131.327462) (xy 214.219487 131.308066) (xy 214.270792 131.2506)
+					(xy 214.333117 131.205513) (xy 214.406461 131.172805) (xy 214.422452 131.167749) (xy 214.355076 131.13839)
+					(xy 214.293524 131.095929) (xy 214.245132 131.042819) (xy 214.208072 130.973439) (xy 214.189126 130.900426)
+					(xy 214.185934 130.856339) (xy 214.454326 130.856339) (xy 214.464284 130.92983) (xy 214.50005 130.995958)
+					(xy 214.50635 131.002885) (xy 214.567807 131.043551) (xy 214.64256 131.057054) (xy 214.648133 131.057107)
+					(xy 214.724517 131.045193) (xy 214.787359 131.006221) (xy 214.790648 131.002885) (xy 214.829666 130.939138)
+					(xy 214.842621 130.862072) (xy 214.842672 130.856339) (xy 214.832715 130.78356) (xy 214.796948 130.718416)
+					(xy 214.790648 130.711625) (xy 214.729008 130.671783) (xy 214.653751 130.658555) (xy 214.648133 130.658503)
+					(xy 214.572903 130.670336) (xy 214.510049 130.709045) (xy 214.506716 130.712358) (xy 214.467424 130.775098)
+					(xy 214.454377 130.85072) (xy 214.454326 130.856339) (xy 214.185934 130.856339) (xy 214.184316 130.833991)
+					(xy 214.190276 130.754786) (xy 214.208158 130.683224) (xy 214.243192 130.610798) (xy 214.293796 130.548356)
+					(xy 214.308879 130.534305) (xy 214.376932 130.48606) (xy 214.445644 130.455152) (xy 214.522911 130.434799)
+					(xy 214.595949 130.425753) (xy 214.648133 130.42403)
 				)
 			)
